Commit message: fix leg linkage mass properties

File: resources/robots/hector_v2/xacro/robot.urdf (robot description, URDF)
Before this commit: robot hector, 30 links, 29 joints
Links:
- link L_calf: mass 0.303 -> 0.14647
- link L_hip: mass 0.224 -> 0.1733
- link L_hip2: mass 0.095 -> 0.072
- link L_thigh: mass 0.642 -> 0.348
- link L_toe: mass 0.214 -> 0.085
- link R_calf: mass 0.303 -> 0.14647
- link R_hip: mass 0.224 -> 0.1733
- link R_hip2: mass 0.095 -> 0.072
- link R_thigh: mass 0.642 -> 0.34806
- link R_toe: mass 0.214 -> 0.08592
- link trunk: mass 4.98 -> 4.8

Commit message: Update com param

File: resources/robots/hector_v2/xacro/robot.urdf (robot description, URDF)
Before this commit: robot hector, 30 links, 29 joints
Links:
- link trunk: mass 4.8 -> 4.78

Commit message: 1st commit

File: resources/robots/hector_v2/xacro/robot.urdf (robot description, URDF)
Before this commit: robot hector, 30 links, 29 joints
Links:
- link L_toe: geometry collision mesh filename=../meshes/Foot.STL scale=1 1 1; visual mesh filename=../meshes/Foot.STL scale=1 1 1
- link R_toe: geometry collision mesh filename=../meshes/Foot.STL scale=1 1 1; visual mesh filename=../meshes/Foot.STL scale=1 1 1

Commit message: update

File: resources/robots/hector_v2/xacro/robot.urdf (robot description, URDF)
Before this commit: robot hector, 30 links, 29 joints
Links:
- link L_thigh: geometry visual mesh filename=../meshes/thigh_combined_L2.stl scale=1 1 1
- link L_toe: geometry collision box size=0.15 0.04 0.02; visual mesh filename=../meshes/Foot.STL scale=1 1 1
- link R_thigh: geometry visual mesh filename=../meshes/thigh_combined_R2.stl scale=1 1 1
- link R_toe: geometry collision box size=0.15 0.04 0.02; visual mesh filename=../meshes/Foot.STL scale=1 1 1

Commit message: update

File: resources/robots/hector_v2/xacro/robot.urdf (robot description, URDF)
Before this commit: robot hector, 30 links, 29 joints
Links:
- link L_toe: geometry collision box size=0.14 0.03 0.02; visual mesh filename=../meshes/Foot.STL scale=1 1 1
- link R_toe: geometry collision box size=0.14 0.03 0.02; visual mesh filename=../meshes/Foot.STL scale=1 1 1

Commit message: add g1

File: resources/robots/hector_v2/xacro/robot.urdf (robot description, URDF)
Before this commit: robot hector, 30 links, 29 joints
Links:
- link R_toe: mass 0.08592 -> 0.085
