Commit message: update wheel leg

File: resources/robots/go2w/urdf/go2w.urdf (robot description, URDF)
Before this commit: robot go2w_description, 33 links, 32 joints
Joints:
- joint FL_foot_joint: type continuous -> revolute
- joint FR_foot_joint: type continuous -> revolute
- joint RL_foot_joint: type continuous -> revolute
- joint RR_foot_joint: type continuous -> revolute
